File: pcb/hotswap/jorian.kicad_sch (KiCad schematic)
At the start: 59 parts, among them J1 USB-C Conn, J2 Ex_Bat, Q1 AO3407, SW1 SW_PUSH, SW10 SW_PUSH, SW11 SW_PUSH, SW12 SW_PUSH, SW13 SW_PUSH, SW14 SW_PUSH, SW15 SW_PUSH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

Commit message: Add files via upload
Parts:
- added P1: CONN_1, xiao-main:gnd pad, symbol conn:CONN_1
- renumbered E5 to E1, E19 to E2, E10 to E3, E20 to E4, E15 to E5, E21 to E6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
Connections:
- net GND: now also P1.1
